Commit message: update

File: assets/urdf/sobit_pro_tray_new.urdf (robot description, URDF)
Before this commit: robot sobit_pro, 69 links, 68 joints
Links:
- link hand_camera_link: geometry visual cylinder length=0.026 radius=0.0305
- link head_camera_base_link: geometry visual mesh filename=/home/sobits/catkin_ws/src/sobit_pro/sobit_pro_description/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 scale=0.001 0.001 0.001
- link head_camera_pan_link: geometry visual mesh filename=/home/sobits/catkin_ws/src/sobit_pro/sobit_pro_description/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 scale=0.001 0.001 0.001
- link head_camera_plug_base_link: geometry visual mesh filename=/home/sobits/catkin_ws/src/azure_kinect_ros_driver/meshes/a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
- link lidar_base_link: geometry visual mesh filename=/home/sobits/catkin_ws/src/sobit_pro/sobit_pro_description/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 scale=0.001 0.001 0.001
- link mic_base_link: geometry visual mesh filename=/home/sobits/catkin_ws/src/sobit_pro/sobit_pro_description/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 scale=0.001 0.001 0.001
- link mic_link: geometry visual mesh filename=/home/sobits/catkin_ws/src/sobit_pro/sobit_pro_description/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 scale=0.001 0.001 0.001
- link plate_bottom_link: mass 2.7779999999999996 -> 75.0; geometry visual mesh filename=/home/sobits/catkin_ws/src/sobit_pro/sobit_pro_description/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 scale=0.001 0.001 0.001
- link plate_middle_link: geometry visual mesh filename=/home/sobits/catkin_ws/src/sobit_pro/sobit_pro_description/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 scale=0.001 0.001 0.001
- link plate_top_link: geometry visual mesh filename=/home/sobits/catkin_ws/src/sobit_pro/sobit_pro_description/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 scale=0.001 0.001 0.001
- link wheel_b_l_steer_base_link: geometry visual mesh filename=/home/sobits/catkin_ws/src/sobit_pro/sobit_pro_description/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 scale=0.001 0.001 0.001
- link wheel_b_l_steer_link: geometry visual mesh filename=/home/sobits/catkin_ws/src/sobit_pro/sobit_pro_description/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 scale=0.001 0.001 0.001
- link wheel_b_r_steer_base_link: geometry visual mesh filename=/home/sobits/catkin_ws/src/sobit_pro/sobit_pro_description/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 scale=0.001 0.001 0.001
- link wheel_b_r_steer_link: geometry visual mesh filename=/home/sobits/catkin_ws/src/sobit_pro/sobit_pro_description/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 scale=0.001 0.001 0.001
- link wheel_f_l_steer_base_link: geometry visual mesh filename=/home/sobits/catkin_ws/src/sobit_pro/sobit_pro_description/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 scale=0.001 0.001 0.001
- link wheel_f_l_steer_link: geometry visual mesh filename=/home/sobits/catkin_ws/src/sobit_pro/sobit_pro_description/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 scale=0.001 0.001 0.001
- link wheel_f_r_steer_base_link: geometry visual mesh filename=/home/sobits/catkin_ws/src/sobit_pro/sobit_pro_description/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 scale=0.001 0.001 0.001
- link wheel_f_r_steer_link: geometry visual mesh filename=/home/sobits/catkin_ws/src/sobit_pro/sobit_pro_description/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 scale=0.001 0.001 0.001

Commit message: update urdf

File: assets/urdf/sobit_pro_tray_new.urdf (robot description, URDF)
Before this commit: robot sobit_pro, 69 links, 68 joints
Links:
- link wheel_b_l_drive_link: mass 0.235 -> 100.0
- link wheel_b_r_drive_link: mass 0.235 -> 100.0
- link wheel_f_l_drive_link: mass 0.235 -> 100.0
- link wheel_f_r_drive_link: mass 0.235 -> 100.0
